File: kicad/spotify-led-matrix.kicad_sch (KiCad schematic)
At the start: 30 parts, among them J1 Conn_01x02, J2 DisplayConnector, J3 DisplayPWR, J4 BOOT, SW1 NowPlaying, SW2 LikedSongs, SW3 SW_Push, SW4 SW_Push, SW5 SW_Push, SW6 RotaryEncoder_Switch, U1 ESP32-WROOM-32E, U2 TLV1117LV33DCYR

Commit message: Added some connections for SPI communication to display
Parts:
- added C6: 0.1uF, symbol Device:C
- added J5: DisplayOutput, symbol Connector_Generic:Conn_01x05
- added J6: UART, symbol Connector_Generic:Conn_01x04
- added J7: JTAG, symbol Connector_Generic:Conn_01x04
- added R9: 0, symbol Device:R
- added SW5: SW_Push, symbol Switch:SW_Push
- D1: value BLINK -> DEV
- J2: value DisplayConnector -> DisplayInput
Connections:
- net LAT is gone; now on net GPIO22: J2.14 (Pin_14)
- net R1 is gone; now on net PI_R1: J2.1 (Pin_1)
- net ~{OE} is gone; now on net GPIO16: J2.15 (Pin_15)
- net +3V3: now also R7.2, J6.1 (Pin_1); no longer R7.1
- net A: now also U1.31 (IO19)
- net B: now also U1.37 (IO23)
- net C: now also U1.30 (IO18)
- net CLK: now also U1.14 (IO12), J7.2 (Pin_2)
- net D: now also U1.29 (IO5)
- net E: now also U1.23 (IO15), J7.4 (Pin_4)
- net GND: now also J4.2 (Pin_2), U1.15 (GND), U1.38 (GND), U1.39 (GND), U1.40 (GND), U1.41 (GND), U1.42 (GND), U1.43 (GND), U1.44 (GND), U1.45 (GND), U1.46 (GND), U1.47 (GND), C6.2, J6.4 (Pin_4), SW5.1; no longer J4.1 (Pin_1)
- net EN: now reaches C5.1, U1.3 (EN)
- net EN: now also R7.1, R9.2; no longer R7.2
- net at U1.25 (IO0): now also J4.1 (Pin_1); no longer J4.2 (Pin_2)
- net TMS: now reaches U1.13 (IO14)
- net TMS: now also J7.1 (Pin_1)
- net PI_R1: now reaches U1.16 (IO13)
- net PI_R1: now also J7.3 (Pin_3)
- net GPIO16: now reaches U1.27 (IO16)
- net RXD0: now reaches U1.34 (IO3)
- net RXD0: now also J6.3 (Pin_3)
- net TXD0: now reaches U1.35 (IO1)
- net TXD0: now also J6.2 (Pin_2)
- net GPIO22: now reaches U1.36 (IO22)
- net B1 renamed PI_B1
- net PI_B1: now also J5.4 (Pin_4)
- net B2 renamed PI_B2
- net PI_B2: now also J5.5 (Pin_5)
- net G1 renamed PI_G1
- net PI_G1: now also J5.2 (Pin_2)
- net G2 renamed PI_G2
- net PI_G2: now also J5.3 (Pin_3)
- net R2 renamed PI_R2
- net PI_R2: now also J5.1 (Pin_1)
- net Switch Function TBD (Mute?) renamed VolumeMute
- new net: C6.1, R9.1, SW5.2
Other:
- note added: "FROM THE PxMatrix LIBRARY ON GITHUB: When driving a long chain of LED modules in a row, parallel color data lines make a lot of sense since it reduces the data rate. But since we are only driving a few modules here, we really don't need that. We can therefore use jumper wires between input connector (PI) and output connector (PO) to chain all shift registers together and create one big shift regi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"
- note added: "If your panel input connector has "R0" in the top left corner, connect PI and PO as follows: PI PO R1 R0 G0 R1 G1 G0 B0 G1 B1 B0"
- note added: "If your panel input connector has "R1" in the top left corner, connect PI and PO as follows: PI PO R2 R1 G1 R2 G2 G1 B1 G2 B2 B1"
- note added: "Pins 39-47 are EPAD located on the bottom of the module. Soldering them to ground is not required, but it can optimize thermal performance."
- note added: "T = RC = 1ms"
- moved on the sheet: C3, C4, C5, D1, J2, J4, R10, R7, R8, RV1, U1

Commit message: Only updated PDF to show the current schematic.
Parts:
- removed J4: BOOT, symbol Connector_Generic:Conn_01x02
- removed J6: UART, symbol Connector_Generic:Conn_01x04
- removed J7: JTAG, symbol Connector_Generic:Conn_01x04
- removed RV1: R_Potentiometer_US, symbol Device:R_Potentiometer_US
- removed SW1: NowPlaying, symbol Switch:SW_Push
- removed SW2: LikedSongs, symbol Switch:SW_Push
- removed SW3, SW4: SW_Push, symbol Switch:SW_Push
- added C10, C12, C7: 0.1uF, symbol Device:C
- added C11: 4.7uF, symbol Device:C
- added C8, C9: 10nF, symbol Device:C
- added D2: MODES, symbol Device:LED
- added D3: BRIGHTNESS, symbol Device:LED
- added D4: VOLUME, symbol Device:LED
- added D5: D, symbol Device:D
- added D6, D8, D9: TODO, Diode_THT:D_P600_R-6_P20.00mm_Horizontal, symbol Diode:5KPxxCA
- added J4: USB, symbol Connector_Generic:Conn_01x04
- added J6: JUMPER, symbol Connector_Generic:Conn_01x03
- added Q2, Q3: SS8050-G, spotify-led-matrix:TRANS_SS8050-G, symbol spotify-led-matrix:SS8050-G
- added R12, R13, R19, R20, R26: 10k, symbol Device:R
- added R14, R15: 22, symbol Device:R
- added R18, R21, R22: 0, symbol Device:R
- added R23: 22.1k, symbol Device:R
- added R24: 47.5k, symbol Device:R
- added R25: 1k, symbol Device:R
- added U3: SN74LVC1G14DBV, Package_TO_SOT_SMD:SOT-23-5, symbol 74xGxx:SN74LVC1G14DBV
- added U4: CP2102N-A01-GQFN28, spotify-led-matrix:QFN50P500X500X80-29N, symbol spotify-led-matrix:CP2102N-A01-GQFN28
- added U5: NVT2003DP_118, spotify-led-matrix:TSSOP10_SOT552-1_NXP, symbol spotify-led-matrix:NVT2003DP_118
- J1: value Conn_01x02 -> +5V_JACK
- J2: value DisplayInput -> PANEL_IN
- J3: value DisplayPWR -> DISPLAY_PWR
- J5: value DisplayOutput -> PANEL_OUT
- R10, R11, R5, R6: value R -> 10k
- R4: value R -> 1k
- SW1: renamed from SW6; value RotaryEncoder_Switch -> SELECT; footprint (none) -> spotify-led-matrix:EVEYBCAJ008B
- SW5: value SW_Push -> BOOT
- SW5: value SW_Push -> EN
- U2: value TLV1117LV33DCYR -> TLV1117LV33DCYR or TLV1117LV
Connections:
- net LikedSongs is gone; now on net +5V: R5.1
- net Mode3 TBD is gone; now on an unnamed net: R4.1
- net +3V3: now also C11.1, C12.1, R25.1, U4.6 (VDD), U4.7 (VREGIN), U5.10 (EN), U5.9 (VREFB); no longer SW1.S2, SW5.1
- net +5V: now also R11.1, J6.2 (Pin_2), R12.1, U3.5 (VCC), U5.2 (VREFA); no longer J1.1 (Pin_1)
- net CLK: no longer J2.13 (Pin_13)
- net EN: now also Q2.3
- net GND: now also SW1.C, SW1.S1, SW5.1, C10.2, C11.2, C12.2, C7.2, C8.2, C9.2, D6.1 (A1), D8.1 (A1), D9.1 (A1), J4.4 (Pin_4), R24.1, R26.2, U3.3 (GND), U4.29 (GND), U4.3 (GND), U5.1 (GND); no longer R10.2, R4.2, R5.2
- net RXD0: now also R22.1
- net TXD0: now also R21.1
- net at R11.2: now also SW1.S2, D5.2 (A)
- net at U1.25 (IO0): now also R14.1, R15.1
- net at SW1.A: now also R12.2, R13.1
- net at SW1.B: now also R10.1, R5.2
- net EnDisplay renamed ENABLE_PWR
- net Mode4 TBD: no longer names the net of R3.1
- net Mode4 TBD: now also D4.1 (K)
- net Mode5 TBD: no longer names the net of R2.1
- net Mode5 TBD: now also D3.1 (K); no longer SW5.2
- net NowPlaying: no longer names the net of R1.1
- net NowPlaying: now also D2.1 (K)
- removed net VolumeMute: R10.1, SW1.S1
- new net: Q2.1, R19.2
- new net: C8.1, R10.2, U5.4 (A2)
- new net: C7.1, D5.1 (K), R4.2, U3.2
- new net: U3.4, U5.3 (A1)
- new net: R23.2, R24.2, U4.8 (VBUS)
- new net: C9.1, R13.2, U5.5 (A3)
- new net: C10.1, R18.1, SW5.2
- new net: R26.1, U4.11 (~{SUSPENDB})
- new net: Q3.1, R20.2
- new net: R25.2, U4.9 (~{RST})
- new net BOOT_BTN: R14.2, R18.2
- new net BOOT_T: Q3.2, R15.2
- new net BRIGHTNESS: D3.2 (A)
- new net D+: D9.2 (A2), J4.3 (Pin_3), U4.4 (D+)
- new net D-: D8.2 (A2), J4.2 (Pin_2), U4.5 (D-)
- new net DTR: Q3.3, R19.1, U4.28 (DTR)
- new net MODES: D2.2 (A)
- new net ROTARY_A: U5.6 (B3)
- new net ROTARY_B: U5.7 (B2)
- new net RTS: Q2.2, R20.1, U4.24 (RTS)
- new net RXD: R21.2, U4.25 (RXD)
- new net SELECT: U5.8 (B1)
- new net TXD: R22.2, U4.26 (TXD)
- new net VBUS: D6.2 (A2), J4.1 (Pin_1), J6.1 (Pin_1), R23.1
- new net VCOM: J1.1 (Pin_1), J6.3 (Pin_3)
- new net VOLUME: D4.2 (A)
- no-connect marks 0 -> 15
Other:
- note added: "+5V will going to the display will carry up to 4A"
- note added: "Auto program DTR RTS -> EN BOOT 0 0 1 1 0 1 1 0 1 0 0 1 1 1 1 1"
- note added: "By connecting the input and output connectors, we create one big shift register, allowing us to use SPI to drive it."
- note added: "CLK, ~{OE}, and LAT are pulled high on the panel."
- note added: "DNP"
- note added: "DNP if using IO0 as CLK"
- note added: "T=RC=1ms"
- note removed: "FROM THE PxMatrix LIBRARY ON GITHUB: When driving a long chain of LED modules in a row, parallel color data lines make a lot of sense since it reduces the data rate. But since we are only driving a few modules here, we really don't need that. We can therefore use jumper wires between input connector (PI) and output connector (PO) to chain all shift registers together and create one big shift regi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"
- note removed: "If your panel input connector has "R0" in the top left corner, connect PI and PO as follows: PI PO R1 R0 G0 R1 G1 G0 B0 G1 B1 B0"
- note removed: "If your panel input connector has "R1" in the top left corner, connect PI and PO as follows: PI PO R2 R1 G1 R2 G2 G1 B1 G2 B2 B1"
- note removed: "Pins 39-47 are EPAD located on the bottom of the module. Soldering them to ground is not required, but it can optimize thermal performance."
- note removed: "T = RC = 1ms"
- moved on the sheet: C1, C2, C3, C4, C5, C6, D1, J1, J2, J3, J5, Q1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

Commit message: Replaced USB to UART converter and updated schematic format
Parts:
- removed D1: DEV, symbol Device:LED
- removed D6, D8, D9: TODO, Diode_THT:D_P600_R-6_P20.00mm_Horizontal, symbol Diode:5KPxxCA
- removed J4: USB, symbol Connector_Generic:Conn_01x04
- removed J6: JUMPER, symbol Connector_Generic:Conn_01x03
- removed Q1: ~, symbol Transistor_FET:DMN2041L
- removed R15: 22, symbol Device:R
- removed U3: SN74LVC1G14DBV, Package_TO_SOT_SMD:SOT-23-5, symbol 74xGxx:SN74LVC1G14DBV
- removed U4: CP2102N-A01-GQFN28, spotify-led-matrix:QFN50P500X500X80-29N, symbol spotify-led-matrix:CP2102N-A01-GQFN28
- removed U5: NVT2003DP_118, spotify-led-matrix:TSSOP10_SOT552-1_NXP, symbol spotify-led-matrix:NVT2003DP_118
- added C1, C2: 47pF, Capacitor_SMD:C_0805_2012Metric_Pad1.18x1.45mm_HandSolder, symbol Device:C
- added C13, C14: 0.1uF, Capacitor_SMD:C_0805_2012Metric, symbol Device:C
- added C3, C4, C5: 100nF, Capacitor_SMD:C_0805_2012Metric_Pad1.18x1.45mm_HandSolder, symbol Device:C
- added C6: 4.7uF, Capacitor_SMD:C_0805_2012Metric_Pad1.18x1.45mm_HandSolder, symbol Device:C_Polarized
- added D11: USB, LED_SMD:LED_0805_2012Metric, symbol Device:LED
- added D12: DEV, LED_SMD:LED_0805_2012Metric, symbol Device:LED
- added D6, D7, D8, D9: D, symbol Device:D
- added J8: USB_Micro-B_Wuerth-629105150521, Connector_USB:USB_Micro-B_Wuerth_629105150521_CircularHoles, symbol picozed-adc:USB_OTG
- added Q1, Q4, Q5, Q6: Q_NMOS_DGS, symbol Device:Q_NMOS_DGS
- added R1, R2: 27, Resistor_SMD:R_0805_2012Metric_Pad1.20x1.40mm_HandSolder, symbol Device:R
- added R16, R27, R29, R30, R35, R36, R37, R38: 10k, Resistor_SMD:R_0805_2012Metric, symbol Device:R
- added R17, R28: 1k, Resistor_SMD:R_0805_2012Metric, symbol Device:R
- added R3: DNP, Resistor_SMD:R_0603_1608Metric, symbol Device:R
- added R39, R40: R, Resistor_SMD:R_0805_2012Metric, symbol Device:R
- added U1: FT234XD-R, spotify-led-matrix:SON45P300X300X80-13N, symbol ilock-test:FT234XD-R
- added U3: MC74HC1G14DTT1G, spotify-led-matrix:SOT95P275X110-5N, symbol spotify-led-matrix:SN74LVC1G14DBV
- added U4: NVT2003DP_118, spotify-led-matrix:TSSOP10_SOT552-1_NXP, symbol spotify-led-matrix:NVT2003DP_118
- added U6, U7: SN74LVC1G14DBV, spotify-led-matrix:SOT95P275X110-5N, symbol spotify-led-matrix:SN74LVC1G14DBV
- C1, C10, C12, C2, C3, C4, C5, C6, C7, C8, C9: footprint (none) -> Capacitor_SMD:C_0805_2012Metric
- C11: value 4.7uF -> 0.1uF; footprint (none) -> Capacitor_SMD:C_0805_2012Metric
- D2, D3, D4: footprint (none) -> LED_SMD:LED_0805_2012Metric
- R1, R10, R12, R13, R14, R18, R19, R2, R20, R21, R22, R3, R5, R6, R7, R9: footprint (none) -> Resistor_SMD:R_0805_2012Metric
- R11, R26: value 10k -> 1k; footprint (none) -> Resistor_SMD:R_0805_2012Metric
- R23: value 22.1k -> 10k; footprint (none) -> Resistor_SMD:R_0805_2012Metric
- R24: value 47.5k -> 1k; footprint (none) -> Resistor_SMD:R_0805_2012Metric
- R25, R4: value 1k -> 10k; footprint (none) -> Resistor_SMD:R_0805_2012Metric
- R8: value R -> 22; footprint (none) -> Resistor_SMD:R_0805_2012Metric
Connections:
- net VCOM is gone; now on net +5V: J1.1 (Pin_1)
- net +3V3: now also R30.1, R36.1, R38.1, U4.10 (EN), U4.9 (VREFB); no longer C11.1, C12.1, R25.1
- net +5V: now also R23.1, R25.1, R4.1, C3.1, C5.1, C6.1, Q1.1 (D), Q4.2 (G), Q5.2 (G), Q6.2 (G), R16.1, R27.1, R29.1, R35.1, R37.1, U1.4 (VCC), U3.5 (VCC), U4.2 (VREFA), U6.5 (VCC), U7.5 (VCC); no longer R11.1
- net BOOT_BTN: now also R8.2; no longer R14.2
- net CLK: now also J2.13 (Pin_13)
- net ENABLE_PWR: now also Q1.2 (G)
- net GND: now also C1.2, C13.2, C14.2, C2.2, C3.2, C4.2, C5.2, C6.2, J8.5 (GND), R3.1, R39.2, R40.2, U1.13 (GND), U1.5 (GND), U3.3 (GND), U4.1 (GND), U6.3 (GND), U7.3 (GND); no longer R24.1, R26.2, R8.2
- net ROTARY_A: now also Q6.3 (S), R38.2, U4.6 (B3)
- net ROTARY_B: now also Q5.3 (S), R36.2, U4.7 (B2)
- net RTS: now also U1.8 (RTS#)
- net RXD: now also U1.10 (RXD)
- net SELECT: now also Q4.3 (S), R30.2, U4.8 (B1)
- net TXD: now also U1.7 (TXD)
- net VBUS: now also D11.2 (A), J8.1 (VBUS); no longer R23.1
- net GPIO0: now reaches R8.1
- net GPIO0: now also R14.1, U1.25 (IO0)
- net at R10.1, R5.2: no longer SW1.B
- net at C7.1, D5.1 (K): now also R11.2, U6.2; no longer R4.2
- net at R24.2: now also C11.1, D6.1 (K); no longer R23.2
- net at R12.2, R13.1: no longer SW1.A
- net at R26.1: now also R25.2, SW1.S2, D8.2 (A)
- net at J3.1 (Pin_1): now also Q1.3 (S)
- net GPIO2: now reaches U1.24 (IO2)
- net GPIO2: now also D12.2 (A)
- net BOOT_T renamed BOOT_AUTO
- net BOOT_AUTO: now also R14.2
- net DTR renamed CTS
- net CTS: now also U1.11 (CTS#)
- new net: C12.1, D8.1 (K), R26.2, U3.2
- new net: C1.1, J8.3 (D+), R1.1
- new net: R1.2, U1.1 (USBDM)
- new net: C4.1, U1.2 (~{RESET}#), U1.3 (3V3OUT), U1.9 (VCCIO)
- new net: C13.1, D7.1 (K), R17.2
- new net: Q5.1 (D), R35.2, U6.4
- new net: D6.2 (A), R23.2, R24.1
- new net: D12.1 (K), R40.1
- new net: D7.2 (A), R16.2, R17.1
- new net: C14.1, D9.1 (K), R28.2, U7.2
- new net: D9.2 (A), R27.2, R28.1, SW1.A
- new net: D11.1 (K), R39.1
- new net: C2.1, J8.2 (D-), R2.1
- new net: R2.2, U1.12 (USBDP)
- new net: D5.2 (A), R11.1, R4.2, SW1.B
- new net: Q4.1 (D), R29.2, U3.4
- new net: Q6.1 (D), R37.2, U7.4
- new net Earth: J8.6 (Shield), R3.2
- no-connect marks 15 -> 1
Other:
- note added: "Auto Program"
- note added: "DISPLAY CONNECTORS"
- note added: "DTR RTS -> EN BOOT 0 0 1 1 0 1 1 0 1 0 0 1 1 1 1 1"
- note added: "Debounce Level Shifters"
- note added: "ESP32 MODULE"
- note added: "LEDS"
- note added: "Manual Program"
- note added: "PROGRAMMING"
- note added: "ROTARY ENCODER CONTROLLER"
- note added: "Series Termination"
- note added: "USB TO UART"
- note added: "VOLTAGE INPUT AND REGULATOR"
- note removed: "Auto program DTR RTS -> EN BOOT 0 0 1 1 0 1 1 0 1 0 0 1 1 1 1 1"
- moved on the sheet: C1, C10, C2, C3, C4, C5, C6, D2, D3, D4, J1, J2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

Commit message: Finished schematic and picked out most parts
Parts:
- removed C11, C13: 0.1uF, Capacitor_SMD:C_0805_2012Metric, symbol Device:C
- removed C8, C9: 10nF, Capacitor_SMD:C_0805_2012Metric, symbol Device:C
- removed D12: DEV, LED_SMD:LED_0805_2012Metric, symbol Device:LED
- removed D6, D7: D, symbol Device:D
- removed J1: +5V_JACK, symbol Connector_Generic:Conn_01x02
- removed J2: PANEL_IN, symbol Connector_Generic:Conn_02x08_Odd_Even
- removed J3: DISPLAY_PWR, symbol Connector_Generic:Conn_01x02
- removed J5: PANEL_OUT, symbol Connector_Generic:Conn_01x05
- removed J8: USB_Micro-B_Wuerth-629105150521, Connector_USB:USB_Micro-B_Wuerth_629105150521_CircularHoles, symbol picozed-adc:USB_OTG
- removed Q1, Q4, Q5, Q6: Q_NMOS_DGS, symbol Device:Q_NMOS_DGS
- removed Q2, Q3: SS8050-G, spotify-led-matrix:TRANS_SS8050-G, symbol spotify-led-matrix:SS8050-G
- removed R13, R23, R37, R38, R5, R6: 10k, Resistor_SMD:R_0805_2012Metric, symbol Device:R
- removed R17, R24: 1k, Resistor_SMD:R_0805_2012Metric, symbol Device:R
- removed R18, R21, R22, R9: 0, Resistor_SMD:R_0805_2012Metric, symbol Device:R
- removed R3, R40: R, Resistor_SMD:R_0805_2012Metric, symbol Device:R
- removed R3: DNP, Resistor_SMD:R_0603_1608Metric, symbol Device:R
- removed U4: NVT2003DP_118, spotify-led-matrix:TSSOP10_SOT552-1_NXP, symbol spotify-led-matrix:NVT2003DP_118
- added D1: BRIGHTNESS, LED_THT:LED_D5.0mm_Horizontal_O1.27mm_Z9.0mm, symbol Device:LED
- added F1: Fuse, Fuse:Fuse_1206_3216Metric_Pad1.42x1.75mm_HandSolder, symbol Device:Fuse
- added J1: +5V, spotify-led-matrix:54-00166, symbol spotify-led-matrix:54-00166
- added J2: DSIPLAY_IN, Connector_PinSocket_2.54mm:PinSocket_2x10_P2.54mm_Vertical, symbol Connector_Generic:Conn_02x10_Odd_Even
- added J3: DISPLAY_PWR, symbol Connector:Screw_Terminal_01x02
- added J4: DISPLAY_OUT, Connector_PinHeader_2.54mm:PinHeader_2x08_P2.54mm_Horizontal, symbol Connector_Generic:Conn_02x08_Odd_Even
- added J5: USB_C_Receptacle_USB2.0, spotify-led-matrix:MOLEX_2169900003, symbol Connector:USB_C_Receptacle_USB2.0
- added Q10, Q4, Q5, Q6, Q7, Q8, Q9: IRLML6244TRPBF, Package_TO_SOT_SMD:SOT-23, symbol Transistor_FET:IRLML6244
- added Q2, Q3: SS8050-G, Package_TO_SOT_SMD:SOT-23-3, symbol Transistor_FET:IRLML6244
- added R15: 120, Resistor_SMD:R_1206_3216Metric_Pad1.30x1.75mm_HandSolder, symbol Device:R
- added R3: 82, Resistor_THT:R_Axial_DIN0207_L6.3mm_D2.5mm_P7.62mm_Horizontal, symbol Device:R
- added R31, R34: 10k, Resistor_SMD:R_1206_3216Metric_Pad1.30x1.75mm_HandSolder, symbol Device:R
- C1, C10, C12, C14, C2, C3, C4, C5, C6, C7, D5, D8, D9: Vendor (none) -> Digikey
- D11: footprint LED_SMD:LED_0805_2012Metric -> LED_THT:LED_D5.0mm_Horizontal_O1.27mm_Z9.0mm; MPN (none) -> WP7113SGC; Manufacturer (none) -> Kingbright; VPN (none) -> 754-1273-ND; Vendor (none) -> Digikey
- D2: footprint LED_SMD:LED_0805_2012Metric -> LED_THT:LED_D5.0mm_Horizontal_O1.27mm_Z9.0mm; MPN (none) -> SSL-LX5093VC; Manufacturer (none) -> Lumex Opto/Components Inc.; VPN (none) -> 67-2064-ND; Vendor (none) -> Digikey
- D3: value BRIGHTNESS -> VOLUME; footprint LED_SMD:LED_0805_2012Metric -> LED_THT:LED_D5.0mm_Horizontal_O1.27mm_Z9.0mm; MPN (none) -> SSL-LX5093VC; Manufacturer (none) -> Lumex Opto/Components Inc.; VPN (none) -> 67-2064-ND; Vendor (none) -> Digikey
- D4: value VOLUME -> DEV; footprint LED_SMD:LED_0805_2012Metric -> LED_THT:LED_D5.0mm_Horizontal_O1.27mm_Z9.0mm; MPN (none) -> WP7113SGC; Manufacturer (none) -> Kingbright; VPN (none) -> 754-1273-ND; Vendor (none) -> Digikey
- R1, R2: footprint Resistor_SMD:R_0805_2012Metric_Pad1.20x1.40mm_HandSolder -> Resistor_SMD:R_1206_3216Metric_Pad1.30x1.75mm_HandSolder; MPN (none) -> RMCF1206FT27R0; Manufacturer (none) -> Stackpole Electronics Inc; VPN (none) -> RMCF1206FT27R0CT-ND; Vendor (none) -> Digikey
- R1, R2: value R -> 82; footprint Resistor_SMD:R_0805_2012Metric -> Resistor_THT:R_Axial_DIN0207_L6.3mm_D2.5mm_P7.62mm_Horizontal; MPN (none) -> RMCF1206FT82R0; Manufacturer (none) -> Stackpole Electronics Inc; VPN (none) -> 738-RMCF1206FT82R0CT-ND; Vendor (none) -> Digikey
- R10, R12: value 10k -> 22; footprint Resistor_SMD:R_0805_2012Metric -> Resistor_SMD:R_1206_3216Metric_Pad1.30x1.75mm_HandSolder; MPN (none) -> RMCF1206FT22R0; Manufacturer (none) -> Stackpole Electronics Inc; VPN (none) -> RMCF1206FT22R0CT-ND; Vendor (none) -> Digikey
- R11, R26, R28: footprint Resistor_SMD:R_0805_2012Metric -> Resistor_SMD:R_1206_3216Metric_Pad1.30x1.75mm_HandSolder; MPN (none) -> RMCF1206FT1K00; Manufacturer (none) -> Stackpole Electronics Inc; VPN (none) -> RMCF1206FT1K00CT-ND; Vendor (none) -> Digikey
- R14, R8: footprint Resistor_SMD:R_0805_2012Metric -> Resistor_SMD:R_1206_3216Metric_Pad1.30x1.75mm_HandSolder; MPN (none) -> RMCF1206FT22R0; Manufacturer (none) -> Stackpole Electronics Inc; VPN (none) -> RMCF1206FT22R0CT-ND; Vendor (none) -> Digikey
- R16: value 10k -> 0; footprint Resistor_SMD:R_0805_2012Metric -> Resistor_SMD:R_1206_3216Metric_Pad1.30x1.75mm_HandSolder; MPN (none) -> RMCF1206FT1R00; Manufacturer (none) -> Stackpole Electronics Inc; VPN (none) -> RMCF1206FT1R00CT-ND; Vendor (none) -> Digikey
- R19, R20, R25, R27, R29, R30, R35, R36, R4, R7: footprint Resistor_SMD:R_0805_2012Metric -> Resistor_SMD:R_1206_3216Metric_Pad1.30x1.75mm_HandSolder; MPN (none) -> RMCF1206FT10K0; Manufacturer (none) -> Stackpole Electronics Inc; VPN (none) -> RMCF1206FT10K0CT-ND; Vendor (none) -> Digikey
- R39: value R -> 120; footprint Resistor_SMD:R_0805_2012Metric -> Resistor_SMD:R_1206_3216Metric_Pad1.30x1.75mm_HandSolder; MPN (none) -> RMCF1206FT120R; Manufacturer (none) -> Stackpole Electronics Inc; VPN (none) -> RMCF1206FT120RCT-ND; Vendor (none) -> Digikey
- SW1: value SELECT -> MODE_SELECT; footprint spotify-led-matrix:EVEYBCAJ008B -> spotify-led-matrix:CUI_ACZ11BR1E-20FD1-20C; MPN (none) -> ACZ11BR1E-20FD1-12C; Manufacturer (none) -> CUI Devices; VPN (none) -> 102-1760-ND; Vendor (none) -> Digikey
- SW5: footprint (none) -> spotify-led-matrix:SW_TL3301DF160QG; MPN (none) -> PTS 647 SK70 SMTR2 LFS; Manufacturer (none) -> C&K; VPN (none) -> PTS647SK70SMTR2LFSCT-ND; Vendor (none) -> Digikey
- U1: MANUFACTURER FTDI -> (none); MAXIMUM_PACKAGE_HEIGHT 0.8mm -> (none); MPN (none) -> FT234XD-R; Manufacturer (none) -> FTDI, Future Technology Devices International Ltd; PARTREV Version 1.2 -> (none); STANDARD IPC-7351B -> (none); VPN (none) -> 768-1178-1-ND; Vendor (none) -> Digikey
- U1: MP ESP32-WROOM-32E -> (none); Manufacturer (none) -> Espressif Systems; Vendor (none) -> Digikey
- U2: value TLV1117LV33DCYR or TLV1117LV -> 5V_TO_3V3; footprint (none) -> Package_TO_SOT_SMD:SOT-223-3_TabPin2; MPN (none) -> TLV1117LV33DCYR; Manufacturer (none) -> Texas Instruments; VPN (none) -> 296-28778-1-ND; Vendor (none) -> Digikey
- U3: footprint spotify-led-matrix:SOT95P275X110-5N -> Package_TO_SOT_SMD:SOT-23-5_HandSoldering; MPN (none) -> MC74HC1G14DTT1G; Manufacturer (none) -> onsemi; VPN (none) -> MC74HC1G14DTT1GOSCT-ND; Vendor (none) -> Digikey
- U6, U7: value SN74LVC1G14DBV -> MC74HC1G14DTT1G; footprint spotify-led-matrix:SOT95P275X110-5N -> Package_TO_SOT_SMD:SOT-23-5_HandSoldering; MPN (none) -> MC74HC1G14DTT1G; Manufacturer (none) -> onsemi; VPN (none) -> MC74HC1G14DTT1GOSCT-ND; Vendor (none) -> Digikey
Connections:
- net BOOT_BTN is gone; now on net BOOT_SW: R8.2
- net RXD is gone; now on net RXD0: U1.10 (RXD)
- net SELECT is gone; now on net +3V3: R30.2
- net TMS is gone; now on net CLK: U1.13 (IO14)
- net TXD is gone; now on net TXD0: U1.7 (TXD)
- net +3V3: now also R35.2, R36.2, U2.2 (OUT); no longer R30.1, R36.1, U2.3 (OUT)
- net +5V: now also R25.2, R27.2, R29.2, R4.2, U2.3 (IN), F1.1, J1.A, Q10.3 (D), Q4.1 (G), Q5.1 (G), Q6.1 (G), Q7.3 (D), Q8.3 (D), Q9.3 (D), R31.2, R34.2; no longer R12.1, R16.1, R25.1, R27.1, R29.1, R35.1, R4.1, U2.1 (IN)
- net BOOT_AUTO: now also Q3.2 (S)
- net BRIGHTNESS: now also U1.28 (IO17), Q8.1 (G); no longer D3.2 (A)
- net CLK: now also J2.15 (Pin_15); no longer U1.14 (IO12)
- net CTS: now also Q3.3 (D)
- net EN: now also R10.1, R12.1
- net GND: now also D11.1 (K), D2.1 (K), D3.1 (K), D4.1 (K), R16.2, U2.1 (GND), D1.1 (K), J1.B, J1.C, J2.18 (Pin_18), J2.6 (Pin_6), J3.2 (Pin_2), J4.16 (Pin_16), J4.4 (Pin_4), J5.A1 (GND), J5.A12 (GND), J5.B1 (GND), J5.B12 (GND); no longer R1.2, R2.2, R39.2, U2.2 (GND)
- net MODES: now also U1.33 (IO21), Q7.1 (G); no longer D2.2 (A)
- net ROTARY_A: now also R36.1, U1.11 (IO26), Q6.3 (D)
- net ROTARY_B: now also R35.1, U1.10 (IO25), Q5.3 (D); no longer R36.2
- net RTS: now also Q2.2 (S)
- net VBUS: now also R39.2, J5.A4 (VBUS), J5.A9 (VBUS), J5.B4 (VBUS), J5.B9 (VBUS); no longer D11.2 (A)
- net VOLUME: now also U1.26 (IO4), Q9.1 (G); no longer D4.2 (A)
- net at R19.2: now also Q2.1 (G)
- net at D8.2 (A), R26.1, SW1.S2: now also R25.1; no longer R25.2
- net at C1.1, R1.1: now also J5.A7 (D-), J5.B7 (D-)
- net at R2.1: now also D1.2 (A); no longer D3.1 (K)
- net at U6.4: now also Q5.2 (S), R31.1; no longer R35.2
- net EN_SW: now reaches C6.1, SW5.2
- net EN_SW: now also R12.2
- net BOOT_SW: now reaches C10.1, SW5.2
- net at D9.2 (A), R28.1, SW1.A: now also R27.1; no longer R27.2
- net at R39.1: now also D11.2 (A); no longer D11.1 (K)
- net at C2.1, R2.1: now also J5.A6 (D+), J5.B6 (D+)
- net EN_AUTO: now reaches R10.2
- net EN_AUTO: now also Q2.3 (D)
- net at D5.2 (A), R11.1, SW1.B: now also R4.1; no longer R4.2
- net at U3.4: now also R29.1, Q4.2 (S); no longer R29.2
- net at U7.4: now also Q6.2 (S), R34.1
- net at R1.1: now also D2.2 (A); no longer D2.1 (K)
- net MODE_SELECT: now reaches U1.9 (IO33)
- net MODE_SELECT: now also R30.1, Q4.3 (D)
- net at R20.2: now also Q3.1 (G)
- net A renamed CS_A
- net CS_A: now also J2.11 (Pin_11)
- net B renamed CS_B
- net CS_B: now also J2.12 (Pin_12)
- net C renamed CS_C
- net CS_C: now also J2.13 (Pin_13)
- net D renamed CS_D
- net CS_D: now also J2.14 (Pin_14)
- net E renamed CS_E
- net CS_E: now also J2.10 (Pin_10)
- net GPIO0 renamed BOOT
- net GPIO16 renamed ~{OE}
- net ~{OE}: now also J2.17 (Pin_17)
- net GPIO2 renamed DEV
- net DEV: now also Q10.1 (G)
- net GPIO22 renamed ~{LAT}
- net PI_R1 renamed R1_IN
- net R1_IN: now also J2.3 (Pin_3)
- new net: D4.2 (A), R15.1
- new net: Q10.2 (S), R15.2
- new net: F1.2, J3.1 (Pin_1)
- new net: Q8.2 (S), R2.2
- new net: Q9.2 (S), R3.2
- new net: J5.S1 (SHIELD), R16.1
- new net: D3.2 (A), R3.1
- new net: Q7.2 (S), R1.2
- new net B1_IN: J2.5 (Pin_5), J4.6 (Pin_6)
- new net B1_OUT: J2.9 (Pin_9), J4.3 (Pin_3)
- new net G1_IN: J2.4 (Pin_4), J4.5 (Pin_5)
- new net G1_OUT: J2.8 (Pin_8), J4.2 (Pin_2)
- new net LAT: J2.16 (Pin_16)
- new net R1_OUT: J2.7 (Pin_7), J4.1 (Pin_1)
- no-connect marks 1 -> 31
Other:
- note added: "(5-2.2)V / 20mA = 140R LEDs are used to show the USB connection while programming and for general development. This could be to show the rotary encoder is working or other thins TBD later."
- note added: "(5-3.2)V / 20mA = 90R LEDs are used to show what mode you are in while turning the rotary encoder."
- note added: "All outputs on the rotary encoder are connected to +5V (high). When turning the encoder or pressing the switch, it pulls them to ground (low). When the rotary encoder is pulled low, the schmitt trigger's output goes high. When the schmitt trigger output goes high, it is then level shifted down to +3V3 so that the ESP32's digital input pins can handle it."
- note added: "By connecting the input and output connectors, we create one big shift register, allowing us to use SPI to drive it. R1_IN internally connects to R1_OUT, and so on."
- note added: "CLK, ~{OE}, and LAT are pulled high on the display's input connector. CLK and LAT are pulled high on the display's output connector. ~{OE} is pulled low on the display's output connector."
- note added: "CTS RTS -> EN BOOT 0 0 1 1 0 1 1 0 1 0 0 1 1 1 1 1"
- note added: "Caps of lower value should go closer to device on the layout."
- note added: "DNP cap if using IO0 as CLK"
- note added: "Debounce Circuits Level Shifters"
- note added: "Display will draw up to 4A; ESP32 will draw up to 500mA. Power jack is rated for 6A and is 2.1mm x 5.5mm"
- note added: "My PCB will screw into the back/side of the display. The DISPLAY_IN connector will plug directly into the display. The DISPLAY_OUT connector will have a ribbon cables the display. The DISPLAY_PWR connector will have a spade to rectangular cable. The DISPLAY_IN connector is 2x10 in order to more snugly fit into the display's 2x08 connector."
- note added: "My inputs: SELECT, ROTARY_B, ROTARY_A My outputs: ENABLE_PWR, MODES, BRIGHTNESS, VOLUME, DEV BOOT and EN are found in the PROGRAMMING circuits. The rest of the connections go to the display's input."
- note added: "NOTE: GPIO 34-39 are input only."
- note added: "POWER INPUT AND REGULATOR"
- note added: "Project by Austin Driggs | Fall 2023"
- note added: "SPOTIFY LED MATRIX"
- note added: "Series Termination Circuits"
- note added: "This can be helpful to "minimize reflections and improve the quality of the signal because it is split in two places"."
- note added: "VBUS serves no purpose and only lights up an LED when plugged in. Connecting the USB shield directly to GND can sometimes cause problems (if the two don't exactly "agree" on what GND is, so a 0R is placed to prevent this issue."
- note removed: "+5V will going to the display will carry up to 4A"
- note removed: "By connecting the input and output connectors, we create one big shift register, allowing us to use SPI to drive it."
- note removed: "CLK, ~{OE}, and LAT are pulled high on the panel."
- note removed: "DNP"
- note removed: "DNP if using IO0 as CLK"
- note removed: "DTR RTS -> EN BOOT 0 0 1 1 0 1 1 0 1 0 0 1 1 1 1 1"
- note removed: "Debounce Level Shifters"
- note removed: "Series Termination"
- note removed: "VOLTAGE INPUT AND REGULATOR"
- moved on the sheet: C1, C10, C12, C14, C2, C3, C4, C5, C6, C7, D11, D2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
