File: kicad/spotify-led-matrix.kicad_sch (KiCad schematic)
At the start: 75 parts, among them J1 +5V, J2 DSIPLAY_IN, J3 DISPLAY_PWR, J4 DISPLAY_OUT, J5 USB_C_Receptacle_USB2.0, Q10 IRLML6244TRPBF, Q2 SS8050-G, Q3 SS8050-G, Q4 IRLML6244TRPBF, Q5 IRLML6244TRPBF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

Commit message: Working out gitignore issues.
Connections:
- new net: SW1.P1, SW1.P2
Changed lines of the file:
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@@
     (stroke (width 0) (type default))
-  )
-  (rectangle (start -519.43 55.88) (end -398.145 207.01)
-    (stroke (width 0) (type default))
-    (fill (type none))
-  )
-  (rectangle (start -384.175 49.53) (end -266.065 166.37)
-    (stroke (width 0) (type default))
-    (fill (type none))
-  )
-  (rectangle (start -499.11 6.35) (end -413.385 51.435)
-    (stroke (width 0) (type default))
-    (fill (type none))
-  )
-  (rectangle (start -245.11 22.86) (end -142.24 109.855)
-    (stroke (width 0) (type default))
-    (fill (type none))
-  )
-  (rectangle (start -379.095 170.815) (end -271.78 260.985)
-    (stroke (width 0) (type default))
-    (fill (type none))
-  )
-  (rectangle (start -238.76 116.205) (end -149.86 222.885)
-    (stroke (width 0) (type default))
-    (fill (type none))
-  )
-  (rectangle (start -521.97 211.455) (end -395.605 273.05)
-    (stroke (width 0) (type default))
-    (fill (type none))
   )
   (text "VBUS serves no purpose and only lights up an LED when plugged in.\n\nConnecting the USB shield directly to GND can sometimes cause problems (if the two \ndon't exactly \"agree\" on what GND is, so a 0R is placed to prevent this issue."
@@
   (symbol (lib_id "Device:RotaryEncoder_Switch") (at 37.465 144.145 180) (unit 1)
     (in_bom yes) (on_board yes) (dnp no) (fields_autoplaced)
-    (property "Reference" "SW1" (at 37.465 134.62 0)
-      (effects (font (size 1.27 1.27)))
-    )
-    (property "Value" "MODE_SELECT" (at 37.465 137.16 0)
-      (effects (font (size 1.27 1.27)))
-    )
-    (property "Footprint" "spotify-led-matrix:CUI_ACZ11BR1E-20FD1-20C" (at 41.275 148.209 0)
-      (effects (font (size 1.27 1.27)) hide)
-    )
-    (property "Datasheet" "https://www.cuidevices.com/product/resource/acz11.pdf" (at 37.465 150.749 0)
-      (effects (font (size 1.27 1.27)) hide)
-    )
-    (property "MPN" "ACZ11BR1E-20FD1-12C" (at 37.465 144.145 0)
-      (effects (font (size 1.27 1.27)) hide)
-    )
-    (property "VPN" "102-1760-ND" (at 37.465 144.145 0)
-      (effects (font (size 1.27 1.27)) hide)
-    )
-    (property "Description" "ROTARY ENCODER INCREMENT 12PPR" (at 37.465 144.145 0)
-      (effects (font (size 1.27 1.27)) hide)
-    )
-    (property "Manufacturer" "CUI Devices" (at 37.465 144.145 0)
-      (effects (font (size 1.27 1.27)) hide)
-    )
-    (property "Vendor" "Digikey" (at 37.465 144.145 0)
+    (property "Reference" "SW1" (at 37.465 152.4 0)
+      (effects (font (size 1.27 1.27)))
+    )
+    (property "Value" "MODE_SELECT" (at 37.465 150.495 0)
+      (effects (font (size 1.27 1.27)))
+    )
+    (property "Footprint" "spotify-led-matrix:CUI_ACZ11BR1E-20FD1-20C" (at 38.1 128.27 0)
+      (effects (font (size 1.27 1.27)) hide)
+    )
+    (property "Datasheet" "https://www.cuidevices.com/product/resource/acz11.pdf" (at 34.29 130.81 0)
+      (effects (font (size 1.27 1.27)) hide)
+    )
+    (property "MPN" "ACZ11BR1E-20FD1-12C" (at 34.29 128.651 0)
+      (effects (font (size 1.27 1.27)) hide)
+    )
+    (property "VPN" "102-1760-ND" (at 34.29 128.651 0)
+      (effects (font (size 1.27 1.27)) hide)
+    )
+    (property "Description" "ROTARY ENCODER INCREMENT 12PPR" (at 34.29 128.651 0)
+      (effects (font (size 1.27 1.27)) hide)
+    )
+    (property "Manufacturer" "CUI Devices" (at 34.29 128.651 0)
+      (effects (font (size 1.27 1.27)) hide)
+    )
+    (property "Vendor" "Digikey" (at 36.83 129.54 0)
       (effects (font (size 1.27 1.27)) hide)
     )
@@
     (pin "B")
     (pin "C")
+    (pin "P2")
+    (pin "P1")
     (pin "S1")
     (pin "S2")
