File: kicad/spotify-led-matrix.kicad_sch (KiCad schematic)
At the start: 75 parts, among them J1 +5V, J2 DSIPLAY_IN, J3 DISPLAY_PWR, J4 DISPLAY_OUT, J5 USB_C_Receptacle_USB2.0, Q10 IRLML6244TRPBF, Q2 SS8050-G, Q3 SS8050-G, Q4 IRLML6244TRPBF, Q5 IRLML6244TRPBF, Q6 IRLML6244TRPBF, Q7 IRLML6244TRPBF, Q8 IRLML6244TRPBF, Q9 IRLML6244TRPBF, SW1 MODE_SELECT, SW5 BOOT, SW5 EN, U1 ESP32-WROOM-32E, U1 FT234XD-R, U2 5V_TO_3V3, U3 MC74HC1G14DTT1G, U6 MC74HC1G14DTT1G, U7 MC74HC1G14DTT1G

Commit message: Cleaned up file organization
Parts:
- removed U3, U6, U7: MC74HC1G14DTT1G, Package_TO_SOT_SMD:SOT-23-5_HandSoldering, symbol spotify-led-matrix:SN74LVC1G14DBV
- added U3, U4, U5: MC74HC1G14DTT1G, Package_TO_SOT_SMD:SOT-23-5_HandSoldering, symbol spotify-led-matrix:MC74HC1G14DTT1G
- J2: value DSIPLAY_IN -> DISPLAY_IN
Connections:
- net +5V: now also U3.5 (VCC), U4.5 (VCC), U5.5 (VCC)
- net GND: now also U3.3 (GND), U4.3 (GND), U5.3 (GND)
- net at C12.1, D8.1 (K), R26.2: now also U3.2
- net at C7.1, D5.1 (K), R11.2: now also U4.2
- net at Q5.2 (S), R31.1: now also U4.4
- net at Q6.2 (S), R34.1: now also U5.4
- net at Q4.2 (S), R29.1: now also U3.4
- net at C14.1, D9.1 (K), R28.2: now also U5.2

Commit message: Cleaned up a lot and started pcb layout
Parts:
- removed C3, C5: 100nF, Capacitor_SMD:C_0805_2012Metric_Pad1.18x1.45mm_HandSolder, symbol Device:C
- removed C3: 22uF, Capacitor_SMD:C_0805_2012Metric, symbol Device:C
- removed C5: 1uF, Capacitor_SMD:C_0805_2012Metric, symbol Device:C
- removed C6: 4.7uF, Capacitor_SMD:C_0805_2012Metric_Pad1.18x1.45mm_HandSolder, symbol Device:C_Polarized
- removed D11: USB, LED_THT:LED_D5.0mm_Horizontal_O1.27mm_Z9.0mm, symbol Device:LED
- removed D8, D9: D, symbol Device:D
- removed J3: DISPLAY_PWR, symbol Connector:Screw_Terminal_01x02
- removed J4: DISPLAY_OUT, Connector_PinHeader_2.54mm:PinHeader_2x08_P2.54mm_Horizontal, symbol Connector_Generic:Conn_02x08_Odd_Even
- removed Q10: IRLML6244TRPBF, Package_TO_SOT_SMD:SOT-23, symbol Transistor_FET:IRLML6244
- removed R39: 120, Resistor_SMD:R_1206_3216Metric_Pad1.30x1.75mm_HandSolder, symbol Device:R
- removed U1: FT234XD-R, spotify-led-matrix:SON45P300X300X80-13N, symbol ilock-test:FT234XD-R
- added C3, C5: 100nF, Capacitor_SMD:C_1206_3216Metric_Pad1.33x1.80mm_HandSolder, symbol Device:C
- added C3: 22uF, Capacitor_SMD:C_1206_3216Metric_Pad1.33x1.80mm_HandSolder, symbol Device:C
- added C3: 4.7uF, Capacitor_SMD:C_1206_3216Metric_Pad1.33x1.80mm_HandSolder, symbol Device:C
- added C5: 1uF, Capacitor_SMD:C_1206_3216Metric_Pad1.33x1.80mm_HandSolder, symbol Device:C
- added D6, D7: D, Diode_SMD:D_SOD-523, symbol Device:D
- added D8: MODES, LED_THT:LED_D5.0mm_Horizontal_O1.27mm_Z9.0mm, symbol Device:LED
- added J3: DISPLAY_PWR, symbol Connector_Generic:Conn_01x04
- added J4: DISPLAY_OUT, Connector_PinSocket_2.54mm:PinSocket_2x10_P2.54mm_Vertical, symbol Connector_Generic:Conn_02x10_Odd_Even
- added Q1: IRLML6244TRPBF, Package_TO_SOT_SMD:SOT-23, symbol Transistor_FET:IRLML6244
- added R13, R17: 1k, Resistor_SMD:R_1206_3216Metric_Pad1.30x1.75mm_HandSolder, symbol Device:R
- added R5: 10k, Resistor_SMD:R_1206_3216Metric_Pad1.30x1.75mm_HandSolder, symbol Device:R
- added R6: 82, Resistor_THT:R_Axial_DIN0207_L6.3mm_D2.5mm_P7.62mm_Horizontal, symbol Device:R
- added R9: 120, Resistor_SMD:R_1206_3216Metric_Pad1.30x1.75mm_HandSolder, symbol Device:R
- added U6: FT231XS-R, spotify-led-matrix:SOP63P599X175-20N, symbol spotify-led-matrix:FT231XS-R
- C1, C10, C12, C14, C2, C4, C6, C7: footprint Capacitor_SMD:C_0805_2012Metric -> Capacitor_SMD:C_1206_3216Metric_Pad1.33x1.80mm_HandSolder
- C1, C2, C4: footprint Capacitor_SMD:C_0805_2012Metric_Pad1.18x1.45mm_HandSolder -> Capacitor_SMD:C_1206_3216Metric_Pad1.33x1.80mm_HandSolder
- D1: value BRIGHTNESS -> USB; footprint LED_THT:LED_D5.0mm_Horizontal_O1.27mm_Z9.0mm -> LED_SMD:LED_0603_1608Metric_Pad1.05x0.95mm_HandSolder; MPN SSL-LX5093VC -> SML-LXFM0603SUGCTR; VPN 67-2064-ND -> 67-2320-1-ND
- D2: value MODES -> DEV; MPN SSL-LX5093VC -> WP7113SGC; Manufacturer Lumex Opto/Components Inc. -> Kingbright; VPN 67-2064-ND -> 754-1273-ND
- D4: value DEV -> BRIGHTNESS; MPN WP7113SGC -> SSL-LX5093VC; Manufacturer Kingbright -> Lumex Opto/Components Inc.; VPN 754-1273-ND -> 67-2064-ND
- D5: footprint (none) -> Diode_SMD:D_SOD-523; MPN (none) -> BAT54XV2T1G; Manufacturer (none) -> onsemi; VPN (none) -> BAT54XV2T1GOSCT-ND
- F1: value Fuse -> 6A
- R1: value 82 -> 120; footprint Resistor_THT:R_Axial_DIN0207_L6.3mm_D2.5mm_P7.62mm_Horizontal -> Resistor_SMD:R_1206_3216Metric_Pad1.30x1.75mm_HandSolder; MPN RMCF1206FT82R0 -> RMCF1206FT120R; VPN 738-RMCF1206FT82R0CT-ND -> RMCF1206FT120RCT-ND
- R15: value 120 -> 1k; MPN RMCF1206FT120R -> RMCF1206FT1K00; VPN RMCF1206FT120RCT-ND -> RMCF1206FT1K00CT-ND
- R16: now not fitted
- R2: value 82 -> 1k; footprint Resistor_THT:R_Axial_DIN0207_L6.3mm_D2.5mm_P7.62mm_Horizontal -> Resistor_SMD:R_1206_3216Metric_Pad1.30x1.75mm_HandSolder; MPN RMCF1206FT82R0 -> RMCF1206FT1K00; VPN 738-RMCF1206FT82R0CT-ND -> RMCF1206FT1K00CT-ND
- R7: value 10k -> 82; footprint Resistor_SMD:R_1206_3216Metric_Pad1.30x1.75mm_HandSolder -> Resistor_THT:R_Axial_DIN0207_L6.3mm_D2.5mm_P7.62mm_Horizontal; MPN RMCF1206FT10K0 -> RMCF1206FT82R0; VPN RMCF1206FT10K0CT-ND -> 738-RMCF1206FT82R0CT-ND
Connections:
- net +3V3: now also C3.1, R5.1; no longer R7.2
- net +5V: now also R3.2, R7.2, C3.1, C3.1, C5.1, R6.2, R9.2, U6.15 (VCC); no longer Q7.3 (D), Q8.3 (D), Q9.3 (D)
- net B1_IN: now also J4.8 (Pin_8)
- net B1_OUT: now also J4.5 (Pin_5)
- net BRIGHTNESS: now also R13.1; no longer Q8.1 (G)
- net DEV: now also R17.1
- net EN: now also C5.1, R5.2; no longer R7.1
- net G1_IN: now also J4.7 (Pin_7)
- net G1_OUT: now also J4.4 (Pin_4)
- net GND: now also Q7.2 (S), Q8.2 (S), Q9.2 (S), C3.2, C3.2, C3.2, C5.2, C5.2, J3.3 (Pin_3), J3.4 (Pin_4), J4.18 (Pin_18), J4.6 (Pin_6), Q1.2 (S), U6.16 (GND), U6.5 (~{RI}), U6.6 (GND), U6.8 (~{DCD}); no longer D2.1 (K), D3.1 (K), D4.1 (K)
- net MODES: now also R15.1; no longer Q7.1 (G)
- net R1_OUT: now also J4.3 (Pin_3)
- net RTS: now also U6.2 (~{RTS})
- net RXD0: now also U6.4 (RXD)
- net TXD0: now also U6.20 (TXD)
- net VBUS: now also R1.2
- net VOLUME: now also R2.1; no longer Q9.1 (G)
- net at R25.1, R26.1, SW1.S2: now also D5.2 (A)
- net at C12.1, R26.2, U3.2: now also D5.1 (K)
- net D+: now reaches C1.1, R1.1
- net D+: now also J5.A6 (D+), J5.B6 (D+); no longer J5.A7 (D-), J5.B7 (D-)
- net USBD+: now reaches R1.2
- net USBD+: now also U6.11 (USBDP)
- net at D4.2 (A): now also R6.1; no longer R15.1
- net at R15.2: now also Q7.1 (G)
- net at F1.2: now also J3.1 (Pin_1), J3.2 (Pin_2)
- net at C4.1: now also U6.13 (3V3OUT), U6.14 (~{RESET}), U6.3 (VCCIO)
- net at C7.1, R11.2, U4.2: now also D6.1 (K); no longer D5.1 (K)
- net at R27.1, R28.1, SW1.A: now also D7.2 (A)
- net at R2.2: now also Q9.1 (G); no longer Q8.2 (S)
- net at C14.1, R28.2, U5.2: now also D7.1 (K)
- net D-: now reaches C2.1, R2.1
- net D-: now also J5.A7 (D-), J5.B7 (D-); no longer J5.A6 (D+), J5.B6 (D+)
- net at R11.1, R4.1, SW1.B: now also D6.2 (A); no longer D5.2 (A)
- net USBD-: now reaches R2.2
- net USBD-: now also U6.12 (USBDM)
- net at D1.2 (A): now also R1.1; no longer R2.1
- net at D2.2 (A): now also R9.1; no longer R1.1
- net CTS renamed DTR
- net DTR: now also U6.1 (~{DTR})
- new net: D3.1 (K), Q9.3 (D)
- new net: D2.1 (K), Q1.3 (D)
- new net: D4.1 (K), Q8.3 (D)
- new net: Q8.1 (G), R13.2
- new net: Q1.1 (G), R17.2
- new net: D8.1 (K), Q7.3 (D)
- new net: D8.2 (A), R7.1
- no-connect marks 31 -> 40
Other:
- note added: "By connecting the input and output connectors, we create one big shift register, allowing us to use SPI to drive it."
- note added: "DTR RTS -> EN BOOT 0 0 1 1 0 1 1 0 1 0 0 1 1 1 1 1"
- note added: "My PCB will screw into the back/side of the display. All connectors will be plugging in directly to the display. The DISPLAY_IN and OUT connectors are 2x10 in order to more snugly fit into the display's 2x08 connector."
- note added: "VBUS serves no purpose and only lights up an LED when plugged in. Connecting the USB shield directly to GND can sometimes cause problems (if the two don't exactly "agree" on what GND is), so a DNP is used to prevent this issue."
- note added: "by Austin Driggs | Fall 2023"
- note removed: "By connecting the input and output connectors, we create one big shift register, allowing us to use SPI to drive it. R1_IN internally connects to R1_OUT, and so on."
- note removed: "CLK, ~{OE}, and LAT are pulled high on the display's input connector. CLK and LAT are pulled high on the display's output connector. ~{OE} is pulled low on the display's output connector."
- note removed: "CTS RTS -> EN BOOT 0 0 1 1 0 1 1 0 1 0 0 1 1 1 1 1"
- note removed: "DNP cap if using IO0 as CLK"
- note removed: "My PCB will screw into the back/side of the display. The DISPLAY_IN connector will plug directly into the display. The DISPLAY_OUT connector will have a ribbon cables the display. The DISPLAY_PWR connector will have a spade to rectangular cable. The DISPLAY_IN connector is 2x10 in order to more snugly fit into the display's 2x08 connector."
- note removed: "My inputs: SELECT, ROTARY_B, ROTARY_A My outputs: ENABLE_PWR, MODES, BRIGHTNESS, VOLUME, DEV BOOT and EN are found in the PROGRAMMING circuits. The rest of the connections go to the display's input."
- note removed: "Project by Austin Driggs | Fall 2023"
- note removed: "VBUS serves no purpose and only lights up an LED when plugged in. Connecting the USB shield directly to GND can sometimes cause problems (if the two don't exactly "agree" on what GND is, so a 0R is placed to prevent this issue."
- moved on the sheet: C1, C10, C2, C4, C6, F1, J5, Q2, Q3, Q7, Q8, Q9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
