File: kicad/spotify-led-matrix.kicad_pcb (KiCad board)
At the start: 2 copper layers, 100.5 x 118 mm, 71 parts, among them J1 +5V, J2 DSIPLAY_IN, J4 DISPLAY_OUT, J5 USB_C_Receptacle_USB2.0, Q10 IRLML6244TRPBF, Q2 SS8050-G, Q3 SS8050-G, Q4 IRLML6244TRPBF, Q5 IRLML6244TRPBF, Q6 IRLML6244TRPBF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

Commit message: Cleaned up a lot and started pcb layout
Parts:
- removed C16, C18: 100nF, Capacitor_SMD:C_0805_2012Metric_Pad1.18x1.45mm_HandSolder
- removed C20: 4.7uF, Capacitor_SMD:C_0805_2012Metric_Pad1.18x1.45mm_HandSolder
- removed D11: USB, LED_THT:LED_D5.0mm_Horizontal_O1.27mm_Z9.0mm
- removed Q10: IRLML6244TRPBF, Package_TO_SOT_SMD:SOT-23
- removed R39: 120, Resistor_SMD:R_1206_3216Metric_Pad1.30x1.75mm_HandSolder
- removed U7: MC74HC1G14DTT1G, Package_TO_SOT_SMD:SOT-23-5_HandSoldering
- removed U8: FT234XD-R, spotify-led-matrix:SON45P300X300X80-13N
- added C11: 100nF, Capacitor_SMD:C_1206_3216Metric_Pad1.33x1.80mm_HandSolder, F.Cu at (112.5, 301.0)
- added C8: 4.7uF, Capacitor_SMD:C_1206_3216Metric_Pad1.33x1.80mm_HandSolder, F.Cu at (112.5, 307.0)
- added C9: 100nF, Capacitor_SMD:C_1206_3216Metric_Pad1.33x1.80mm_HandSolder, F.Cu at (112.5, 304.0)
- added D5: D, Diode_SMD:D_SOD-523, F.Cu at (116.0, 348.0)
- added D6: D, Diode_SMD:D_SOD-523, F.Cu at (168.9, 338.1)
- added D7: D, Diode_SMD:D_SOD-523, F.Cu at (168.7, 359.5)
- added D8: MODES, LED_THT:LED_D5.0mm_Horizontal_O1.27mm_Z9.0mm, F.Cu at (222.4, 307.0)
- added Q1: IRLML6244TRPBF, Package_TO_SOT_SMD:SOT-23, F.Cu at (187.1, 303.5)
- added R13: 1k, Resistor_SMD:R_1206_3216Metric_Pad1.30x1.75mm_HandSolder, F.Cu at (206.5, 301.0)
- added R17: 1k, Resistor_SMD:R_1206_3216Metric_Pad1.30x1.75mm_HandSolder, F.Cu at (183.5, 301.0)
- added R5: 10k, Resistor_SMD:R_1206_3216Metric_Pad1.30x1.75mm_HandSolder, F.Cu at (76.5, 273.8)
- added R6: 82, Resistor_SMD:R_1206_3216Metric_Pad1.30x1.75mm_HandSolder, F.Cu at (214.0, 302.9)
- added R9: 120, Resistor_SMD:R_1206_3216Metric_Pad1.30x1.75mm_HandSolder, F.Cu at (191.0, 303.0)
- added U4: MC74HC1G14DTT1G, Package_TO_SOT_SMD:SOT-23-5_HandSoldering, F.Cu at (176.4, 339.6)
- added U5: MC74HC1G14DTT1G, Package_TO_SOT_SMD:SOT-23-5_HandSoldering, F.Cu at (176.8, 360.6)
- C1, C10, C12, C14, C2, C3, C4, C5, C6, C7: footprint Capacitor_SMD:C_0805_2012Metric -> Capacitor_SMD:C_1206_3216Metric_Pad1.33x1.80mm_HandSolder
- C17, C19, C21: footprint Capacitor_SMD:C_0805_2012Metric_Pad1.18x1.45mm_HandSolder -> Capacitor_SMD:C_1206_3216Metric_Pad1.33x1.80mm_HandSolder
- D1: value BRIGHTNESS -> USB; footprint LED_THT:LED_D5.0mm_Horizontal_O1.27mm_Z9.0mm -> LED_SMD:LED_0603_1608Metric_Pad1.05x0.95mm_HandSolder
- D2: value MODES -> DEV
- D4: value DEV -> BRIGHTNESS
- F1: value Fuse -> 6A
- J2: value DSIPLAY_IN -> DISPLAY_IN
- J4: footprint Connector_PinHeader_2.54mm:PinHeader_2x08_P2.54mm_Horizontal -> Connector_PinSocket_2.54mm:PinSocket_2x10_P2.54mm_Vertical
- R1: value 82 -> 120
- R15: value 120 -> 1k
- R2: value 82 -> 1k
- R7: value 10k -> 82
- U6: value MC74HC1G14DTT1G -> FT231XS-R; footprint Package_TO_SOT_SMD:SOT-23-5_HandSoldering -> spotify-led-matrix:SOP63P599X175-20N
- moved J5 287.5 mm to (95.5, 317.5)
- moved Q2 279.4 mm to (101.6, 324.6), turned to 90 degrees
- moved R34 278.4 mm to (182.0, 359.6), turned to 90 degrees
- moved R28 276.8 mm to (167.4, 362.5)
- moved R27 275.4 mm to (165.5, 358.1), turned to 90 degrees
- moved Q3 274.7 mm to (106.0, 324.6), turned to 90 degrees
- moved R36 272.6 mm to (191.5, 358.6), turned to 90 degrees
- moved R26 270.6 mm to (114.5, 351.5)
- moved R25 269.1 mm to (113.0, 346.6), turned to 90 degrees
- moved C14 267.8 mm to (172.5, 363.6), turned to -90 degrees
- moved Q6 267.4 mm to (186.6, 360.5)
- moved R11 267.2 mm to (167.3, 342.1)
- moved Q4 267.0 mm to (132.5, 349.0)
- moved R31 266.8 mm to (181.4, 338.1), turned to 90 degrees
- moved C12 266.1 mm to (119.5, 351.0), turned to -90 degrees
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Connections:
- C17 pad 1: Net-(C17-Pad1) -> /D+
- C19 pad 1: Net-(C19-Pad1) -> /D-
- C21 pad 1: Net-(U8-3V3OUT) -> Net-(U6-3V3OUT)
- C7 pad 1: Net-(D5-K) (its old number) -> Net-(D6-K)
- D2 pad 1: GND -> Net-(D2-K)
- D3 pad 1: GND -> Net-(D3-K)
- D4 pad 1: GND -> Net-(D4-K)
- J4 pad 1: /R1_OUT -> unconnected-(J4-Pin_1-Pad1)
- J4 pad 16: GND -> unconnected-(J4-Pin_16-Pad16)
- J4 pad 2: /G1_OUT -> unconnected-(J4-Pin_2-Pad2)
- J4 pad 3: /B1_OUT -> /R1_OUT
- J4 pad 4: GND -> /G1_OUT
- J4 pad 5: /G1_IN -> /B1_OUT
- J4 pad 6: /B1_IN -> GND
- J4 pad 7: unconnected-(J4-Pin_7-Pad7) -> /G1_IN
- J4 pad 8: unconnected-(J4-Pin_8-Pad8) -> /B1_IN
- J5 pad A6: Net-(C19-Pad1) -> /D+
- J5 pad A7: Net-(C17-Pad1) -> /D-
- J5 pad B6: Net-(C19-Pad1) -> /D+
- J5 pad B7: Net-(C17-Pad1) -> /D-
- Q3 pad 3: /CTS -> /DTR
- Q7 pad 1: /MODES -> Net-(Q7-G)
- Q7 pad 2: Net-(Q7-S) -> GND
- Q7 pad 3: +5V -> Net-(D8-K)
- Q8 pad 1: /BRIGHTNESS -> Net-(Q8-G)
- Q8 pad 2: Net-(Q8-S) -> GND
- Q8 pad 3: +5V -> Net-(D4-K)
- Q9 pad 1: /VOLUME -> Net-(Q9-G)
- Q9 pad 2: Net-(Q9-S) -> GND
- Q9 pad 3: +5V -> Net-(D3-K)
- R1 pad 1: Net-(D2-A) -> Net-(D1-A)
- R1 pad 2: Net-(Q7-S) -> VBUS
- R11 pad 2: Net-(D5-K) (its old number) -> Net-(D6-K)
- R15 pad 1: Net-(D4-A) -> /MODES
- R15 pad 2: Net-(Q10-S) -> Net-(Q7-G)
- R19 pad 1: /CTS -> /DTR
- R2 pad 1: Net-(D1-A) -> /VOLUME
- R2 pad 2: Net-(Q8-S) -> Net-(Q9-G)
- R3 pad 2: Net-(Q9-S) -> +5V
- R32 pad 1: Net-(C17-Pad1) -> /D+
- R32 pad 2: Net-(U8-USBDM) -> /USBD+
- R33 pad 1: Net-(C19-Pad1) -> /D-
- R33 pad 2: Net-(U8-USBDP) -> /USBD-
- R7 pad 1: /EN -> Net-(D8-A)
- R7 pad 2: +3V3 -> +5V
- U6 pad 1: unconnected-(U6-NC-Pad1) -> /DTR
- U6 pad 2: Net-(D5-K) (its old number) -> /RTS
- U6 pad 3: GND -> Net-(U6-3V3OUT)
- U6 pad 4: Net-(Q5-S) -> /RXD0
- U6 pad 5: +5V -> GND
Other:
- board size 100.5 x 118 mm -> 192.1 x 264.1 mm
- board text added: "Spotify LED Matrix"
- board text added: "by Austin Driggs | Fall 2023"
