File: hardware/spotify-led-matrix.kicad_sch (KiCad schematic)
At the start: 79 parts, among them J1 +5V, J2 DISPLAY_IN, J3 DISPLAY_PWR, J4 DISPLAY_OUT, J5 USB_C_Receptacle_USB2.0, Q1 IRLML6244TRPBF, Q2 SS8050-G, Q3 SS8050-G, Q4 IRLML6244TRPBF, Q5 IRLML6244TRPBF, Q6 IRLML6244TRPBF, Q7 IRLML6244TRPBF, Q8 IRLML6244TRPBF, Q9 IRLML6244TRPBF, SW1 MODE_SELECT, SW5 BOOT, SW5 EN, U1 ESP32-WROOM-32E, U2 5V_TO_3V3, U3 MC74HC1G14DTT1G, U4 MC74HC1G14DTT1G, U5 MC74HC1G14DTT1G, U6 FT231XS-R

Commit message: Reorganized files again: Wanted to push to backup everything.
Parts:
- added TP1: TestPoint, symbol Connector:TestPoint
Changed lines of the file:
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@@
-    (stroke (width 0) (type default))
-  )
-  (wire (pts (xy 191.77 125.73) (xy 203.835 125.73))
     (stroke (width 0) (type default))
   )
@@
         )
       )
+    )
+  )
+  (symbol (lib_id "Connector:TestPoint") (at 130.175 33.02 0) (unit 1)
+    (in_bom yes) (on_board yes) (dnp no)
+    (property "Reference" "TP1" (at 128.27 27.94 0)
+      (effects (font (size 1.27 1.27)) (justify left))
+    )
+    (property "Value" "TestPoint" (at 132.715 30.988 0)
+      (effects (font (size 1.27 1.27)) (justify left) hide)
+    )
+    (property "Footprint" "" (at 135.255 33.02 0)
+      (effects (font (size 1.27 1.27)) hide)
+    )
+    (property "Datasheet" "~" (at 135.255 33.02 0)
+      (effects (font (size 1.27 1.27)) hide)
+    )
+    (pin "1")
+    (instances
+      (project "spotify-led-matrix"
+        (path "/e8265119-8dca-4f29-8463-0c95468306bc"
+          (reference "TP1") (unit 1)
+        )
+      )

Commit message: update
Other:
- note added: "Minimizes reflections and improves the quality of the signal because it is split in two places."
- note removed: "This can be helpful to "minimize reflections and improve the quality of the signal because it is split in two places"."
Changed lines of the file:
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@@
   )
   (text "VBUS serves no purpose and only lights up an LED when plugged in.\n\nConnecting the USB shield directly to GND can sometimes cause problems (if the two \ndon't exactly \"agree\" on what GND is), so a DNP is used to prevent this issue."
-    (at 55.245 280.67 0)
+    (at 55.245 281.94 0)
     (effects (font (size 1.27 1.27)) (justify left bottom))
   )
@@
     (effects (font (size 1.27 1.27)) (justify left bottom))
   )
-  (text "This can be helpful to \"minimize reflections and improve \nthe quality of the signal because it is split in two places\"."
-    (at 185.42 271.145 0)
+  (text "Minimizes reflections and improves the quality of\nthe signal because it is split in two places."
+    (at 191.77 268.605 0)
     (effects (font (size 1.27 1.27)) (justify left bottom))
   )
@@
   (symbol (lib_id "spotify-led-matrix:ESP32-WROOM-32E") (at 222.885 114.3 0) (unit 1)
     (in_bom yes) (on_board yes) (dnp no)
-    (property "Reference" "U1" (at 221.615 111.76 0)
+    (property "Reference" "U1" (at 220.98 111.76 0)
       (effects (font (size 1.27 1.27)) (justify left))
     )

Commit message: worked on the layout
Parts:
- added TP2: +3V3, symbol Connector:TestPoint
- added TP3: GND, symbol Connector:TestPoint
- TP1: value TestPoint -> +5V
Connections:
- net +3V3: now also TP2.1
- net +5V: now also TP1.1
- net GND: now also TP3.1
- no-connect marks 40 -> 41
Other:
- note added: "POWER INPUT AND LDO REGULATOR"
- note removed: "POWER INPUT AND REGULATOR"
- moved on the sheet: C3, C4, J1, TP1

Commit message: layout stuff and .gitignore update
Parts:
- removed C1, C2: 1uF, Capacitor_SMD:C_1206_3216Metric_Pad1.33x1.80mm_HandSolder, symbol Device:C
- removed TP1: +5V, symbol Connector:TestPoint
- removed TP2: +3V3, symbol Connector:TestPoint
- removed TP3: GND, symbol Connector:TestPoint
- removed U2: 5V_TO_3V3, Package_TO_SOT_SMD:SOT-223-3_TabPin2, symbol Regulator_Linear:uA7805
- added TP4: +5V, symbol Connector:TestPoint
- added TP5: GND, symbol Connector:TestPoint
- added TP6: +3V3, symbol Connector:TestPoint
Connections:
- net +3V3: now also TP6.1
- net +5V: now also TP4.1
- net GND: now also TP5.1
- no-connect marks 41 -> 42
Other:
- note added: "POWER INPUT AND REGULATOR"
- note removed: "POWER INPUT AND LDO REGULATOR"
- moved on the sheet: J1

Commit message: backup
Parts:
- R1, R10, R11, R12, R13, R14, R15, R16, R17, R19, R2, R20, R25, R26, R27, R28, R29, R3, R30, R31, R34, R35, R36, R4, R5, R6, R7, R8, R9: symbol Device:R -> Device:R_US
- TP4, TP5, TP6: footprint (none) -> TestPoint:TestPoint_Loop_D2.54mm_Drill1.5mm_Beaded
Other:
- moved on the sheet: J1, TP4, TP5, TP6

Commit message: update
Other:
- note added: "Decoupling Caps of lower value should go closer to device on the layout."
- note removed: "Caps of lower value should go closer to device on the layout."
Changed lines of the file:
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@@
     (effects (font (size 1.27 1.27)) (justify left bottom))
   )
-  (text "NOTE: GPIO 34-39\nare input only." (at 163.195 131.445 0)
+  (text "NOTE: GPIO 34-39\nare input only." (at 159.385 134.62 0)
     (effects (font (size 1.27 1.27)) (justify left bottom))
   )
@@
     (effects (font (size 2.54 2.54) bold) (justify left bottom))
   )
-  (text "Caps of lower value\nshould go closer to\ndevice on the layout."
-    (at 161.29 116.205 0)
+  (text "Decoupling Caps of lower value should\ngo closer to device on the layout."
+    (at 153.035 145.415 0)
     (effects (font (size 1.27 1.27)) (justify left bottom))
   )

Commit message: reformatted schematic and changed parts: - added new voltage regulator: 1117 adjustable (jellybean) - added temp/volt/cur sensor LTC2990 - changed usb to uart IC to SSOP20 footprint - created and added the display connector symbols
Parts:
- removed TP5: GND, TestPoint:TestPoint_Loop_D2.54mm_Drill1.5mm_Beaded, symbol Connector:TestPoint
- removed TP6: +3V3, TestPoint:TestPoint_Loop_D2.54mm_Drill1.5mm_Beaded, symbol Connector:TestPoint
- added C1, C2: 10uF, Capacitor_SMD:C_1206_3216Metric_Pad1.33x1.80mm_HandSolder, symbol Device:C
- added C13: 470pF, Capacitor_SMD:C_1206_3216Metric_Pad1.33x1.80mm_HandSolder, symbol Device:C
- added C15: 0.1uF, Capacitor_SMD:C_1206_3216Metric_Pad1.33x1.80mm_HandSolder, symbol Device:C
- added Q10: MMBT3904, Package_TO_SOT_SMD:SOT-23, symbol Transistor_BJT:MMBT3904
- added R18, R21: ~, Resistor_SMD:R_1206_3216Metric_Pad1.30x1.75mm_HandSolder, symbol Device:R_US
- added R22: 1m, Resistor_SMD:R_1206_3216Metric_Pad1.30x1.75mm_HandSolder, symbol Device:R_US
- added R23, R24: 4.7k, Resistor_SMD:R_1206_3216Metric_Pad1.30x1.75mm_HandSolder, symbol Device:R_US
- added TP1: +5V, TestPoint:TestPoint_Loop_D2.54mm_Drill1.5mm_Beaded, symbol Connector:TestPoint
- added TP2, TP3: GND, TestPoint:TestPoint_Loop_D2.54mm_Drill1.5mm_Beaded, symbol Connector:TestPoint
- added U2: NCP1117-ADJ, Package_TO_SOT_SMD:SOT-223-3_TabPin2, symbol Regulator_Linear:NCP1117-ADJ_SOT223
- added U7: LTC2990, Package_SO:MSOP-10_3x3mm_P0.5mm, symbol Sensor:LTC2990
- J4: symbol Connector_Generic:Conn_02x10_Odd_Even -> spotify-led-matrix:CONN_LED_MATRIX_DISPLAY
- TP4: value +5V -> GND
- U6: footprint spotify-led-matrix:SOP63P599X175-20N -> Package_SO:SSOP-20_3.9x8.7mm_P0.635mm
Connections:
- net +3V3: now also C2.1, R18.2, TP3.1, U2.2 (VO)
- net +5V: now also C1.1, C15.1, R22.2, R23.2, R24.2, TP1.1, U2.3 (VI), U7.1 (V1), U7.10 (VCC); no longer F1.1, TP4.1
- net GND: now also C1.2, C15.2, C2.2, R21.1, TP2.1, U7.5 (GND), U7.8 (ADR0), U7.9 (ADR1)
- net MODE_SELECT: now also U1.10 (IO25); no longer U1.9 (IO33)
- net ROTARY_A: now also U1.12 (IO27); no longer U1.11 (IO26)
- net ROTARY_B: now also U1.11 (IO26); no longer U1.10 (IO25)
- net OSC_IN: now reaches U1.8 (IO32)
- net CLK renamed SPI_CLK
- net SPI_CLK: now also R24.1
- new net: R18.1, R21.2, U2.1 (ADJ)
- new net: C13.1, Q10.1 (B), Q10.3 (C), U7.3 (V3)
- new net: C13.2, Q10.2 (E), U7.4 (V4)
- new net +5VL: F1.1, R22.1, TP4.1, U7.2 (V2)
- new net I2C_CLK: U7.7 (SCL)
- new net I2C_SDA: R23.1, U7.6 (SDA)
- new net OSC_OUT: U1.9 (IO33)
- no-connect marks 42 -> 41
Other:
- note added: "DISPLAY CONNECTORS AND IC MONITER"
- note added: "Full Handshake"
- note added: "USER LEDS"
- note added: "User Program"
- note added: "t=RC=10ms"
- note removed: "DISPLAY CONNECTORS"
- note removed: "LEDS"
- note removed: "Manual Program"
- note removed: "T=RC=1ms"
- moved on the sheet: C1, C10, C2, C3, C4, C5, C6, D1, D2, D3, D4, D8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
