File: hardware/spotify-led-matrix.kicad_sch (KiCad schematic)
At the start: 92 parts, among them J1 +5V, J2 DISPLAY_IN, J3 DISPLAY_PWR, J4 DISPLAY_OUT, J5 USB_C_Receptacle_USB2.0, Q1 IRLML6244TRPBF, Q10 MMBT3904, Q2 SS8050-G, Q3 SS8050-G, Q4 IRLML6244TRPBF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

Commit message: lots of changes: working on finalizing everything!
Parts:
- removed C13: 470pF, Capacitor_SMD:C_1206_3216Metric_Pad1.33x1.80mm_HandSolder, symbol Device:C
- removed C15: 0.1uF, Capacitor_SMD:C_1206_3216Metric_Pad1.33x1.80mm_HandSolder, symbol Device:C
- removed F1: 6A, Fuse:Fuse_1206_3216Metric_Pad1.42x1.75mm_HandSolder, symbol Device:Fuse
- removed Q10: MMBT3904, Package_TO_SOT_SMD:SOT-23, symbol Transistor_BJT:MMBT3904
- removed R22: 1m, Resistor_SMD:R_1206_3216Metric_Pad1.30x1.75mm_HandSolder, symbol Device:R_US
- removed R23, R24: 4.7k, Resistor_SMD:R_1206_3216Metric_Pad1.30x1.75mm_HandSolder, symbol Device:R_US
- removed U7: LTC2990, Package_SO:MSOP-10_3x3mm_P0.5mm, symbol Sensor:LTC2990
- added TP5: EN, TestPoint:TestPoint_Pad_D2.0mm, symbol Connector:TestPoint
- J2: symbol Connector_Generic:Conn_02x10_Odd_Even -> spotify-led-matrix:CONN_LED_MATRIX_DISPLAY
- J5: symbol Connector:USB_C_Receptacle_USB2.0 -> spotify-led-matrix:USB_C_Receptacle_USB2.0
- Q2, Q3: footprint Package_TO_SOT_SMD:SOT-23-3 -> Package_TO_SOT_SMD:SOT-23
- TP1, TP2: footprint TestPoint:TestPoint_Loop_D2.54mm_Drill1.5mm_Beaded -> TestPoint:TestPoint_Pad_D2.0mm
- TP3: value GND -> +3V3; footprint TestPoint:TestPoint_Loop_D2.54mm_Drill1.5mm_Beaded -> TestPoint:TestPoint_Pad_D2.0mm
- TP4: value GND -> BOOT; footprint TestPoint:TestPoint_Loop_D2.54mm_Drill1.5mm_Beaded -> TestPoint:TestPoint_Pad_D2.0mm
Connections:
- net LAT is gone; now on net ~{LAT}: J2.16 (LAT)
- net +5VL: now also J3.1 (Pin_1), J3.2 (Pin_2); no longer TP4.1
- net BOOT: now also TP4.1
- net EN: now also TP5.1
- net B1_OUT renamed B2_IN
- net G1_OUT renamed G2_IN
- net MODE_SELECT renamed BUTTON
- net R1_IN renamed SPI_SDA
- net R1_OUT renamed R2_IN
- no-connect marks 41 -> 34
Other:
- note added: "DISPLAY CONNECTORS"
- note added: "IO2 is generally used as the blink pin"
- note removed: "All outputs on the rotary encoder are connected to +5V (high). When turning the encoder or pressing the switch, it pulls them to ground (low). When the rotary encoder is pulled low, the schmitt trigger's output goes high. When the schmitt trigger output goes high, it is then level shifted down to +3V3 so that the ESP32's digital input pins can handle it."
- note removed: "DISPLAY CONNECTORS AND IC MONITER"
- moved on the sheet: C12, C14, C7, D5, D6, D7, J2, J3, J4, Q4, Q5, Q6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

Commit message: update?
Parts:
- added R22, R23: 22, Resistor_SMD:R_1206_3216Metric_Pad1.30x1.75mm_HandSolder, symbol Device:R_US
Connections:
- net +5VL is gone; now on net +5V: J3.1 (Pin_1), J3.2 (Pin_2)
- net BOOT_AUTO: now also R8.2; no longer R14.2
- net BOOT_SW: now also R14.2; no longer R8.2
- net EN_AUTO: now also R12.2; no longer R10.2
- net EN_SW: now also R10.2; no longer R12.2
- net SPI_CLK: now also R22.2; no longer U1.13 (IO14)
- net SPI_SDA: now also R23.2; no longer U1.16 (IO13)
- new net: R22.1, U1.13 (IO14)
- new net: R23.1, U1.16 (IO13)
Other:
- note added: "Termination resistors are used to...and the resistor value can be increased or decreased as necessary."
- moved on the sheet: R10, R12, R14, R8
